File: Hardware/I2CRJ45X32.brd (EAGLE design)
At the start: 286 x 58 mm, 120 parts, among them IC1 MCP23017SO, IC2 MCP23017SO, IC3 MCP23017SO, IC4 MCP23017SO, IC5 MCP23017SO, IC6 MCP23017SO, IC7 MCP23017SO, IC8 MCP23017SO, J1 I2C-BREAKOUT, J10 I2C Addr 4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

Commit message: Final tweaks and DRC for v3.0.1 release.
Routing:
- net !RESET: track 309.9 -> 308.4 mm
Other:
- board text added: "SKU: I2CRJ45X32"
- board text added: "v3.0.1"
- board text added: "www.superhouse.tv/i2crj45"
- board text removed: "SKU: I2CRJ45X24"
- board text removed: "v3.0"
- board text removed: "www.superhouse.tv/i2crj45x32"
Changed lines of the file:
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@@
 </layers>
 <board>
-<fusionsync huburn="a.cGVyc29uYWw6dWUyZDliZmNi" projecturn="a.cGVyc29uYWw6dWUyZDliZmNiIzIwMTkwMzE1MTgyMjY5OTA2" f3durn="urn:adsk.wipprod:dm.lineage:DjYxxdFGQRSJkThAhwTjww" pcbguid="746883ea-e62c-42e9-9679-e6d9048e007c" lastpulledtime="" lastsyncedchangeguid="1491f9b9-a179-9c0a-9821-19275fe4b9b0" latestrevisionid="8a223982-5d78-40eb-8f6c-1acb446a08da" lastsyncedrevisionid="8a223982-5d78-40eb-8f6c-1acb446a08da" lastboardhashguid="e88fd704-65e3-ad2c-951b-ebae28f650db" lastpushedtime="2021-09-02T23:04:57Z" linktopcb3d="true"/>
+<fusionsync huburn="a.cGVyc29uYWw6dWUyZDliZmNi" projecturn="a.cGVyc29uYWw6dWUyZDliZmNiIzIwMTkwMzE1MTgyMjY5OTA2" f3durn="urn:adsk.wipprod:dm.lineage:DjYxxdFGQRSJkThAhwTjww" pcbguid="" lastpulledtime="" lastsyncedchangeguid="1491f9b9-a179-9c0a-9821-19275fe4b9b0" latestrevisionid="8a223982-5d78-40eb-8f6c-1acb446a08da" lastsyncedrevisionid="8a223982-5d78-40eb-8f6c-1acb446a08da" lastboardhashguid="e88fd704-65e3-ad2c-951b-ebae28f650db" lastpushedtime="2021-09-02T23:04:57Z" linktopcb3d="true"/>
 <plain>
 <wire x1="3" y1="0" x2="0" y2="3" width="0" layer="20" curve="-90"/>
@@
 <wire x1="286" y1="3" x2="283" y2="0" width="0" layer="20" curve="-90"/>
 <wire x1="283" y1="0" x2="3" y2="0" width="0" layer="20"/>
-<text x="1" y="2" size="1.9" layer="21" font="vector" ratio="17">v3.0</text>
-<text x="107.455" y="54.854" size="1.6764" layer="21" font="vector" ratio="17" align="bottom-center">www.superhouse.tv/i2crj45x32</text>
+<text x="0.5" y="3" size="1.4224" layer="21" font="vector" ratio="17">v3.0.1</text>
+<text x="107.455" y="54.854" size="1.6764" layer="21" font="vector" ratio="17" align="bottom-center">www.superhouse.tv/i2crj45</text>
 <hole x="143" y="8" drill="3.2"/>
 <hole x="143" y="50" drill="3.2" locked="yes"/>
@@
 <text x="0.59" y="25.3" size="1.778" layer="21" font="vector" ratio="18" rot="SR0" align="center-left">I2CBR</text>
 <text x="278.09" y="25.3" size="1.778" layer="21" font="vector" ratio="18" rot="SR0" align="center-left">I2CBR</text>
-<text x="37.455" y="1.854" size="2.3" layer="22" font="vector" ratio="17" rot="MR0" align="bottom-center">www.superhouse.tv/i2crj45x32</text>
-<text x="23.191" y="55.171" size="1.4224" layer="22" font="vector" ratio="17" rot="MR0">SKU: I2CRJ45X24</text>
+<text x="37.455" y="1.854" size="2.3" layer="22" font="vector" ratio="17" rot="MR0" align="bottom-center">www.superhouse.tv/i2crj45</text>
+<text x="23.191" y="55.171" size="1.4224" layer="22" font="vector" ratio="17" rot="MR0">SKU: I2CRJ45X32</text>
 <text x="10" y="45.3" size="1.27" layer="21" font="vector" ratio="17" align="bottom-center">RST P/U</text>
 <dimension x1="287" y1="58" x2="287" y2="0" x3="290" y3="29" textsize="1.778" layer="47"/>
@@
 <contactref element="J8" pad="3"/>
 <contactref element="J8" pad="1"/>
-<wire x1="279.75" y1="27.75" x2="279.7" y2="27.8" width="0.3048" layer="1"/>
 <wire x1="23.27" y1="52.54" x2="23.27" y2="50" width="0.3048" layer="16"/>
 <wire x1="23.27" y1="50" x2="23.27" y2="47.46" width="0.3048" layer="16"/>
@@
 <wire x1="202.675" y1="28.6" x2="203.4" y2="28.6" width="0.3048" layer="1"/>
 <wire x1="203.4" y1="28.6" x2="204" y2="28" width="0.3048" layer="1"/>
-<wire x1="202.13" y1="19.95" x2="202.18" y2="20" width="0.3048" layer="16"/>
 <wire x1="202.13" y1="19.95" x2="202.13" y2="26.13" width="0.3048" layer="16"/>
 <wire x1="202.13" y1="26.13" x2="204" y2="28" width="0.3048" layer="16"/>
@@
 <contactref element="IC5" pad="18"/>
 <contactref element="IC6" pad="18"/>
-<wire x1="280.73" y1="36.54" x2="281.46" y2="36.54" width="0.3048" layer="16"/>
-<wire x1="281.46" y1="36.54" x2="278.5" y2="39.5" width="0.3048" layer="16"/>
 <via x="192" y="40" extent="1-16" drill="0.5"/>
 <wire x1="192" y1="40" x2="189.3" y2="40" width="0.3048" layer="1"/>
@@
 <wire x1="160" y1="40" x2="122" y2="40" width="0.254" layer="16"/>
 <wire x1="160" y1="40" x2="192" y2="40" width="0.254" layer="16"/>
-<wire x1="278.5" y1="39.5" x2="278" y2="40" width="0.254" layer="16"/>
-<wire x1="278" y1="40" x2="262" y2="40" width="0.254" layer="16"/>
 <wire x1="262" y1="40" x2="230" y2="40" width="0.254" layer="16"/>
 <wire x1="230" y1="40" x2="192" y2="40" width="0.254" layer="16"/>
@@
 <wire x1="230" y1="40" x2="227.3" y2="40" width="0.3048" layer="1"/>
 <wire x1="227.3" y1="40" x2="227.22" y2="40.08" width="0.3048" layer="1"/>
+<wire x1="277.27" y1="40" x2="280.73" y2="36.54" width="0.254" layer="16"/>
+<wire x1="262" y1="40" x2="277.27" y2="40" width="0.254" layer="16"/>
 </signal>
 <signal name="N$7">
